File: FrequencySensor/FrequencySensor.kicad_sch (KiCad schematic)
At the start: 4 parts

Commit message: Created PCB
Parts:
- removed D?: D_Bridge_+-AA, symbol Device:D_Bridge_+-AA
- added BR1: MP1010G-G, HVDBR:DIP1270W130P1270L1905H780Q4N, symbol HVDBR:MP1010G-G
- added D1: BZV55B3V3, Diode_SMD:D_MiniMELF, symbol Diode:BZV55B3V3
- added J1: Conn_01x02_Male, Connector_Molex:Molex_Mega-Fit_76829-0002_2x01_P5.70mm_Vertical, symbol Connector:Conn_01x02_Male
- 1k1: renamed from 1k; footprint (none) -> Resistor_THT:R_Axial_DIN0204_L3.6mm_D1.6mm_P1.90mm_Vertical
- 39k1: renamed from 39k; footprint (none) -> Resistor_THT:R_Axial_DIN0204_L3.6mm_D1.6mm_P1.90mm_Vertical
- gave numbers to parts that had none: 1
Connections:
- net 120AV: now also BR1.1 (+)
- net 3.3AV: now also D1.1 (K)
- net AGND: now also BR1.3 (-), D1.2 (A)
- new net AC_In1: BR1.2 (~{_1}), J1.2 (Pin_2)
- new net AC_In2: BR1.4 (~{_2}), J1.1 (Pin_1)
Other:
- moved on the sheet: 1k1, 39k1
